Commit message: Basic ros2_control-gazebo integration

File: src/fulmen_description/urdf/config.urdf.xacro (robot description, xacro)
@@ -19,7 +19,34 @@
     <xacro:property name="side_wheel_mass" value="0.5" />
     <xacro:property name="caster_wheel_radius" value="0.05" />
-    <xacro:property name="caster_wheel_mass" value="0.0" />
+    <xacro:property name="caster_wheel_mass" value="0.1" />
     <xacro:property name="lidar_radius" value="0.1" />
     <xacro:property name="lidar_length" value="0.05" />
     <xacro:property name="lidar_mass" value="0.1" />
+    <xacro:macro name="box_inertia" params="mass x y z o_xyz o_rpy">
+        <inertial>
+            <mass value="${mass}" />
+            <origin xyz="${o_xyz}" rpy="${o_rpy}" />
+            <inertia ixx="${(mass/12) * (y*y + z*z)}" ixy="0" ixz="0"
+                     iyy="${(mass/12) * (x*x + z*z)}" iyz="0"
+                     izz="${(mass/12) * (x*x + y*y)}" />
+        </inertial>
+    </xacro:macro>
+    <xacro:macro name="cylinder_inertia" params="mass r l o_xyz o_rpy">
+        <inertial>
+            <mass value="${mass}" />
+            <origin xyz="${o_xyz}" rpy="${o_rpy}" />
+            <inertia ixx="${(mass/12) * (3*r*r + l*l)}" ixy="0" ixz="0"
+                     iyy="${(mass/12) * (3*r*r + l*l)}" iyz="0"
+                     izz="${(mass/2) * (r*r)}" />
+        </inertial>
+    </xacro:macro>
+    <xacro:macro name="sphere_inertia" params="mass r o_xyz o_rpy">
+        <inertial>
+            <mass value="${mass}" />
+            <origin xyz="${o_xyz}" rpy="${o_rpy}" />
+            <inertia ixx="${(2/5) * mass*r*r}" ixy="0" ixz="0"
+                     iyy="${(2/5) * mass*r*r}" iyz="0"
+                     izz="${(2/5) * mass*r*r}" />
+        </inertial>
+    </xacro:macro>
 </robot>

File: src/fulmen_description/urdf/robot.urdf.xacro (robot description, xacro)
@@ -23,4 +23,11 @@
             <material name="grey" />
         </visual>
+        <collision>
+            <geometry>
+                <box size="${base_length} ${base_width} ${base_height}" />
+            </geometry>
+            <origin xyz="0 0 ${base_height/2}" rpy="0 0 0" />
+        </collision>
+        <xacro:box_inertia mass="${base_mass}" x="${base_length}" y="${base_width}" z="${base_height}" o_xyz="0 0 ${base_height/2}" o_rpy="0 0 0" />
     </link>
     <joint name="${base_joint_name}" type="fixed">
@@ -38,4 +45,11 @@
             <material name="white" />
         </visual>
+        <collision>
+            <geometry>
+                <sphere radius="${side_wheel_radius}" />
+            </geometry>
+            <origin xyz="0 0 0" rpy="${-pi/2} 0 0" />
+        </collision>
+        <xacro:cylinder_inertia mass="${side_wheel_mass}" r="${side_wheel_radius}" l="${side_wheel_length}" o_xyz="0 0 0" o_rpy="${-pi/2} 0 0"/>
     </link>
     <joint name="${left_wheel_joint_name}" type="continuous">
@@ -54,4 +68,11 @@
             <material name="white" />
         </visual>
+        <collision>
+            <geometry>
+                <sphere radius="${side_wheel_radius}" />
+            </geometry>
+            <origin xyz="0 0 0" rpy="${-pi/2} 0 0" />
+        </collision>
+        <xacro:cylinder_inertia mass="${side_wheel_mass}" r="${side_wheel_radius}" l="${side_wheel_length}" o_xyz="0 0 0" o_rpy="${-pi/2} 0 0"/>
     </link>
     <joint name="${right_wheel_joint_name}" type="continuous">
@@ -70,4 +91,11 @@
             <material name="white" />
         </visual>
+        <collision>
+            <geometry>
+                <sphere radius="${caster_wheel_radius}" />
+            </geometry>
+            <origin xyz="0 0 0" rpy="0 0 0" />
+        </collision>
+        <xacro:sphere_inertia mass="${caster_wheel_mass}" r="${caster_wheel_radius}" o_xyz="0 0 0" o_rpy="0 0 0" />
     </link>
     <joint name="${caster_wheel_joint_name}" type="fixed">
@@ -85,4 +113,11 @@
             <material name="red" />
         </visual>
+        <collision>
+            <geometry>
+                <cylinder radius="${lidar_radius}" length="${lidar_length}" />
+            </geometry>
+            <origin xyz="0 0 0" rpy="0 0 0" />
+        </collision>
+        <xacro:cylinder_inertia mass="${lidar_mass}" r="${lidar_radius}" l="${lidar_length}" o_xyz="0 0 0" o_rpy="0 0 0" />
     </link>
     <joint name="${lidar_joint_name}" type="fixed">
